Commit message: Adding Lidar

File: src/car_description/src/urdf/car.xacro (robot description, xacro)
@@ -19,5 +19,5 @@
      </xacro:macro>
     <!-- #### chassis property #### -->
-    <xacro:property name="chassis_length" value="0.3"/>
+    <xacro:property name="chassis_length" value="0.65"/>
     <xacro:property name="chassis_width" value="0.3"/>
     <xacro:property name="chassis_height" value="0.05"/>
@@ -26,5 +26,5 @@
     <xacro:property name="caster_length" value="0.015"/>
     <xacro:property name="caster_mass" value="0.2"/>
-    <!-- #####  caster macro   ##### -->
+    <!-- #####  caster macro  ##### -->
     <xacro:macro name="caster" params= "prefix suffix X1 X2 Y1 Y2">
       <joint name="${prefix}_${suffix}_caster_joint" type="fixed">
@@ -145,5 +145,5 @@
       </inertial>
   </link>
-<!-- #### 4 casters  #### -->
+<!-- #### 4 casters #### -->
   <xacro:caster prefix="right" suffix="front" X1="0" X2="1" Y1="-1" Y2="0" />
   <xacro:caster prefix="right" suffix="back" X1="-1" X2="0" Y1="-1" Y2="0"/>
@@ -151,38 +151,20 @@
   <xacro:caster prefix="left" suffix="back" X1="-1" X2="0" Y1="0" Y2="1"/>
 <!-- #### Sensors : Lidar #### -->
-  <joint name="scan_joint1" type="fixed">
-    <parent link="chassis"/>
-    <child link="scan_lidar"/>
-    <!-- <origin xyz="${chassis_length/2-0.03} ${chassis_width/2-0.03} 0.16" rpy="0 0 -${PI/2}"/> -->
-    <origin xyz="0 0 0.16" rpy="0 0 0"/>
-  </joint>
-  <link name="scan_lidar">
-    <visual>
-      <origin xyz="0 0 -.06" rpy="${PI/2} 0 0"/>
-      <geometry>
-        <mesh filename="package://car_description/src/meshes/sensors/hokuyo_lidar.stl" scale="0.012 0.012 0.012"/>
-      </geometry>
-      <material name="black"/>
-    </visual>
-    <collision>
-      <origin xyz="0 0 -.03" rpy="0 0 0"/>
-      <geometry>
-        <cylinder length="0.08" radius="0.025"/>
-      </geometry>
-    </collision>
-    <inertial>
-      <mass value="0.114" />
-      <origin xyz="0 0 0" />
-      <inertia ixx="0.001" ixy="0.0" ixz="0.0"
-               iyy="0.001" iyz="0.0"
-               izz="0.001" />
-    </inertial>
-  </link>
-  <gazebo>
-    <plugin name="gazebo_ros_control" filename="libgazebo_ros_control.so">
-      <robotSimType>gazebo_ros_control/DefaultRobotHWSim</robotSimType>
-      <legacyModeNS>true</legacyModeNS>
-    </plugin>
-  </gazebo>
+<!-- #####    END   ##### -->
+<!-- #####  A1 PART ##### -->
+<!-- #####    END   ##### -->
+<gazebo>
+  <plugin name="gazebo_ros_control" filename="libgazebo_ros_control.so">
+    <robotSimType>gazebo_ros_control/DefaultRobotHWSim</robotSimType>
+    <legacyModeNS>true</legacyModeNS>
+  </plugin>
+</gazebo>
+<!-- #####   BEGIN  ##### -->
+<!-- #####  A2 PART ##### -->
+<!-- #####   BEGIN  ##### -->
+<!-- #####    END   ##### -->
+<!-- #####  A2 PART ##### -->
+<!-- #####    END   ##### -->
 <!-- Begin of camera -->
+<!-- End of camera -->
 </robot>

File: src/car_description/src/urdf/car_gazebo.xacro (robot description, xacro)
@@ -1,5 +1,5 @@
 <?xml version="1.0"?>
 <robot name="$(arg robotName)" xmlns:xacro="http://ros.org/wiki/xacro">
-  <xacro:arg name="laser_visual"  default="false"/>
+  <xacro:arg name="laser_visual"  default="true"/>
   <xacro:arg name="camera_visual" default="false"/>
   <xacro:arg name="imu_visual"    default="false"/>
@@ -9,5 +9,5 @@
   <gazebo reference="wheel_left_link">
     <mu1>10</mu1>
-    <mu2>1</mu2>
+    <mu2>10</mu2>
     <kp>50000.0</kp>
     <kd>10.0</kd>
@@ -19,5 +19,5 @@
   <gazebo reference="wheel_right_link">
     <mu1>10</mu1>
-    <mu2>1</mu2>
+    <mu2>10</mu2>
     <kp>50000.0</kp>
     <kd>10.0</kd>
@@ -59,3 +59,35 @@
     </plugin>
   </gazebo>
+  <gazebo reference="scan_lidar">
+    <material>Gazebo/FlatBlack</material>
+    <sensor type="ray" name="scan_lidar">
+      <pose>0 0 0 0 0 0</pose>
+      <visualize>$(arg laser_visual)</visualize>
+      <update_rate>10</update_rate>
+      <ray>
+        <scan>
+          <horizontal>
+            <samples>725</samples>
+            <resolution>1</resolution>
+            <min_angle>-1.570796</min_angle>
+            <max_angle>1.570796</max_angle>
+          </horizontal>
+        </scan>
+        <range>
+          <min>0.10</min>
+          <max>1.0</max>
+          <resolution>0.01</resolution>
+        </range>
+        <noise>
+          <type>gaussian</type>
+          <mean>0.0</mean>
+          <stddev>0.05</stddev>
+        </noise>
+      </ray>
+      <plugin name="gazebo_ros_lds_lfcd_controller" filename="libgazebo_ros_laser.so">
+        <topicName>scan_lidar</topicName>
+        <frameName>scan_lidar</frameName>
+      </plugin>
+    </sensor>
+  </gazebo>
 </robot>
