Commit message: adding imu

File: src/car_description/src/urdf/carA.xacro (robot description, xacro)
@@ -185,4 +185,32 @@
     </plugin>
   </gazebo>
+<!-- Sensors : IMU -->
+  <joint name="imu_joint" type="fixed">
+      <parent link="chassis"/>
+      <child link="imu_link"/>
+      <origin xyz="0 0 0" rpy="0 0 0"/>
+  </joint>
+  <link name="imu_link">
+    <!-- <visual>
+      <origin xyz="0 0 0" rpy="0 0 0"/>
+      <geometry>
+        <mesh filename="package://car_description/src/meshes/sensors/hokuyo_lidar.stl" scale="0.012 0.012 0.012"/>
+      </geometry>
+      <material name="black"/>
+    </visual> -->
+    <!-- <collision>
+      <origin xyz="0 0 -.03" rpy="0 0 0"/>
+      <geometry>
+        <cylinder length="0.08" radius="0.025"/>
+      </geometry>
+    </collision>
+    <inertial>
+      <mass value="0.114" />
+      <origin xyz="0 0 0" />
+      <inertia ixx="0.001" ixy="0.0" ixz="0.0"
+               iyy="0.001" iyz="0.0"
+               izz="0.001" />
+    </inertial> -->
+  </link>
 <!-- Begin of camera -->
 </robot>

File: src/car_description/src/urdf/car_gazebo.xacro (robot description, xacro)
@@ -91,3 +91,38 @@
     </sensor>
   </gazebo>
+  <gazebo reference="imu_link">
+    <sensor type="imu" name="imu">
+      <always_on>true</always_on>
+      <visualize>$(arg imu_visual)</visualize>
+    </sensor>
+    <material>Gazebo/Grey</material>
+  </gazebo>
+  <gazebo>
+    <plugin name="imu_plugin" filename="libgazebo_ros_imu.so">
+      <alwaysOn>true</alwaysOn>
+      <bodyName>imu_link</bodyName>
+      <frameName>imu_link</frameName>
+      <topicName>imu</topicName>
+      <serviceName>imu_service</serviceName>
+      <gaussianNoise>0.0</gaussianNoise>
+      <updateRate>200</updateRate>
+      <imu>
+        <noise>
+          <type>gaussian</type>
+          <rate>
+            <mean>0.0</mean>
+            <stddev>2e-4</stddev>
+            <bias_mean>0.0000075</bias_mean>
+            <bias_stddev>0.0000008</bias_stddev>
+          </rate>
+          <accel>
+            <mean>0.0</mean>
+            <stddev>1.7e-2</stddev>
+            <bias_mean>0.1</bias_mean>
+            <bias_stddev>0.001</bias_stddev>
+          </accel>
+        </noise>
+      </imu>
+    </plugin>
+  </gazebo>
 </robot>

Commit message: bad day

File: src/car_description/src/urdf/carA.xacro (robot description, xacro)
@@ -165,10 +165,10 @@
       <material name="black"/>
     </visual>
-    <collision>
+    <!-- <collision>
       <origin xyz="0 0 -.03" rpy="0 0 0"/>
       <geometry>
         <cylinder length="0.08" radius="0.025"/>
       </geometry>
-    </collision>
+    </collision> -->
     <inertial>
       <mass value="0.114" />

Commit message: update carA urdf

File: src/car_description/src/urdf/carA.xacro (robot description, xacro)
@@ -21,5 +21,5 @@
     <xacro:property name="chassis_length" value="0.3"/>
     <xacro:property name="chassis_width" value="0.3"/>
-    <xacro:property name="chassis_height" value="0.05"/>
+    <xacro:property name="chassis_height" value="0.1"/>
     <!-- ####  caster property #### -->
     <xacro:property name="caster_radius" value="0.025"/>
@@ -69,5 +69,5 @@
   <link name="chassis">
     <visual>
-      <origin xyz="0.0 0 0.075" rpy="0 0 0"/>
+      <origin xyz="0.0 0 0.1" rpy="0 0 0"/>
       <geometry>
         <box size="${chassis_length} ${chassis_width} ${chassis_height}"/>
@@ -76,5 +76,5 @@
     </visual>
     <collision>
-      <origin xyz="0.0 0 0.075" rpy="0 0 0"/>
+      <origin xyz="0.0 0 0.1" rpy="0 0 0"/>
       <geometry>
         <box size="${chassis_length} ${chassis_width} ${chassis_height}"/>
@@ -155,5 +155,5 @@
     <child link="scan_lidar"/>
     <!-- <origin xyz="${chassis_length/2-0.03} ${chassis_width/2-0.03} 0.16" rpy="0 0 -${PI/2}"/> -->
-    <origin xyz="0 0 0.16" rpy="0 0 0"/>
+    <origin xyz="0 0 0.21" rpy="0 0 0"/>
   </joint>
   <link name="scan_lidar">
